File: Rocket.kicad_sch (KiCad schematic)
At the start: 6 parts, among them U1 BMP280, U2 MPU-6050, U3 ArduinoMicroSD, U4 NEO_6M, U5 FT232RL

Commit message: second commit: update
Connections:
- net at U2.23 (SCL): now also A1.5 (D2); no longer A1.6 (D3)
- net at U2.24 (SDA): now also A1.6 (D3)
- net at U2.9 (AD0): no longer A1.5 (D2)
- net at U3.1 (CS): now also A1.11 (D8)
- net at U3.2 (SCK): now also A1.16 (SCK)
- net at U3.3 (MOSI): now also A1.15 (MISO); no longer A1.8 (D5)
- net at U3.4 (MISO): now also A1.14 (MOSI); no longer A1.7 (D4)
- net at U5.1 (TXD): now also A1.7 (D4); no longer A1.11 (D8)
- net at U5.5 (RXD): now also A1.8 (D5); no longer A1.12 (D9)
- removed net GND: U2.18 (GND), U4.12 (GND), U4.13 (GND), U4.24 (GND)
Other:
- moved on the sheet: A1, U1, U2, U3, U4, U5

Commit message: thrid commit: carried
Parts:
- removed A1: Arduino_Nano_Every, Module:Arduino_Nano, symbol MCU_Module:Arduino_Nano_Every
- removed U1: BMP280, symbol Rocket_Library:BMP280
- removed U2: MPU-6050, Sensor_Motion:InvenSense_QFN-24_4x4mm_P0.5mm, symbol Sensor_Motion:MPU-6050
- removed U3: ArduinoMicroSD, symbol Rocket_Library:ArduinoMicroSD
- removed U4: NEO_6M, symbol Rocket_Library:NEO_6M
- removed U5: FT232RL, Package_SO:SSOP-28_5.3x10.2mm_P0.65mm, symbol Interface_USB:FT232RL
- added A1: Arduino_Nano_v3.x, Module:Arduino_Nano, symbol MCU_Module:Arduino_Nano_v3.x
- added BT1: Battery, symbol Device:Battery
- added C1, C2: C, symbol Device:C
- added U1: ArduinoMicroSD, symbol Rocket_Library:ArduinoMicroSD
- added U2: MPU6050, symbol Rocket_Library:MPU6050
- added U3: Xbee_Apater, symbol Rocket_Library:Xbee_Apater
- added U4: BMP280, symbol Rocket_Library:BMP280
- added U5: NEO_6M, symbol Rocket_Library:NEO_6M
- added U6: L7805, symbol Regulator_Linear:L7805
Connections:
- new net: BT1.1 (+), C1.1, U6.1 (IN)
- new net +5V: A1.27 (+5V), C2.1, U2.1 (VCC), U6.3 (OUT)
- new net CS: A1.13 (D10), U1.1 (CS)
- new net D0: A1.2 (D0/RX), U3.2 (RX)
- new net D1: A1.1 (D1/TX), U3.3 (TX)
- new net D2: A1.5 (D2), U5.2 (RX)
- new net D3: A1.6 (D3), U5.3 (TX)
- new net GND: A1.29 (GND), A1.4 (GND), BT1.2 (-), C1.2, C2.2, U1.6 (GND), U2.2 (GND), U3.4 (GND), U6.2 (GND)
- new net MISO: A1.15 (D12), U1.4 (MISO)
- new net MOSI: A1.14 (D11), U1.3 (MOSI)
- new net SCL: A1.7 (D4), U2.3 (SCL), U4.2 (SCL)
- new net SDA: A1.8 (D5), U2.4 (SDA), U4.3 (SDA)
- new net VCC: U1.5 (VCC), U3.5 (5V), U4.1 (VCC), U5.1 (VCC)
